Commit message: controll of robot via gazebo diff_drive plugin

File: quadruped/robot.urdf.xacro (robot description, xacro)
@@ -10,4 +10,5 @@
         <xacro:include filename="gazebo_control.xacro" />
     </xacro:unless> -->
+    <xacro:include filename="gazebo_control.xacro" />
     <!-- <xacro:include filename="lidar.xacro" /> -->
     <!-- <xacro:include filename="camera.xacro" /> -->

File: quadruped/robot.xacro (robot description, xacro)
@@ -2,5 +2,16 @@
 <robot xmlns:xacro="http://www.ros.org/wiki/xacro" >
 <!-- <robot name="quadruped"> -->
+    <!-- BASE LINK -->
     <link name="base_link">
+    </link>
+    <!-- BASE_FOOTPRINT LINK -->
+    <joint name="base_footprint_joint" type="fixed">
+        <parent link="base_link"/>
+        <child link="base_footprint"/>
+        <origin xyz="0 0 0" rpy="0 0 0"/>
+    </joint>
+    <link name="base_footprint">
+    </link>
+    <link name="base">
         <visual>
             <origin xyz="0.0049215742833825515401 0.008362597111257197291 -0.010279088801785209867" rpy="0 -0 0" />
@@ -24,7 +35,12 @@
         </inertial>
     </link>
-    <gazebo reference="base_link">
+    <gazebo reference="base">
         <material>Gazebo/Orange</material>
     </gazebo>
+    <joint name="base_joint" type="fixed">
+        <parent link="base_link"/>
+        <child link="base"/>
+        <origin xyz="0 0 0" rpy="0 0 0"/>
+    </joint>
     <link name="ball_caster">
         <visual>
@@ -51,8 +67,10 @@
     <gazebo reference="ball_caster">
         <material>Gazebo/White</material>
+        <mu1 value="0.001"/>
+        <mu2 value="0.001"/>
     </gazebo>
     <joint name="link_front_ball" type="fixed">
         <origin xyz="-0.0028254257166174471388 -0.12663740288874275608 -0.010279088801785209867" rpy="0 -0 0" />
-        <parent link="base_link" />
+        <parent link="base" />
         <child link="ball_caster" />
         <axis xyz="0 0 1"/>
@@ -84,8 +102,10 @@
     <gazebo reference="ball_caster_2">
         <material>Gazebo/White</material>
+        <mu1 value="0.001"/>
+        <mu2 value="0.001"/>
     </gazebo>
     <joint name="link_back_ball" type="fixed">
         <origin xyz="-0.0028254257166174540777 0.14336259711125715066 -0.010279088801785206397" rpy="-1.0408340855860799426e-16 5.9887421101386484724e-31 -1.9721522630525262292e-31" />
-        <parent link="base_link" />
+        <parent link="base" />
         <child link="ball_caster_2" />
         <axis xyz="0 0 1"/>
@@ -172,5 +192,5 @@
         <parent link="dc_motor" />
         <child link="wheel" />
-        <axis xyz="0 0 1"/>
+        <axis xyz="0 0 -1"/>
         <limit effort="1" velocity="20" />
         <joint_properties friction="0.0"/>
@@ -186,5 +206,5 @@
     <joint name="link_right_bracket" type="fixed">
         <origin xyz="-0.12367842571661746831 0.0083625971112572007604 -0.0022790888017852097003" rpy="3.141592653589793116 5.1885812976927455838e-73 -1.570796326794896558" />
-        <parent link="base_link" />
+        <parent link="base" />
         <child link="motor_bracket" />
         <axis xyz="0 0 1"/>
@@ -285,5 +305,5 @@
     <joint name="link_left_bracket" type="fixed">
         <origin xyz="0.13352157428338257139 0.0083625971112572007604 -0.0022790888017852097003" rpy="3.141592653589793116 5.1885812976927455838e-73 1.570796326794896558" />
-        <parent link="base_link" />
+        <parent link="base" />
         <child link="motor_bracket_2" />
         <axis xyz="0 0 1"/>
